File: Free_EMS_Board_ruzki.kicad_pcb (KiCad board)
At the start: 2 copper layers, 59.1 x 37.7 mm, 40 parts, among them IC1 MCP2551-I/SN, P1 CONN_20X2_MS, P2 CONN_2, P3 CONN_3X2, U1 MC9S12XDP512, X1 16Mhz

Commit message: ground stitching ..
added some ground stitching, moved c4 and c5 to be closer to the mcu,
moved some components references, added a notch for orientation,
preparation done for PCB manufacturing
Parts:
- PWM3  PWM1: renamed from P2
- moved C4 1.97 mm to (199.2, 111.1)
- moved C5 1.69 mm to (196.6, 110.0)
- renumbered P3 to BDM, JP1 to Load
Routing:
- net GND: track 374.2 -> 492.2 mm, vias 29 -> 47
Other:
- board text added: "v0.3"
